File: NASA Motherboard V4.kicad_pcb (KiCad board)
At the start: 6 copper layers, 200 x 150 mm, 140 parts, among them J101 Screw_Terminal_01x02, J102 Screw_Terminal_01x02, J103 Screw_Terminal_01x02, J104 Screw_Terminal_01x02, J105 Screw_Terminal_01x02, J106 Screw_Terminal_01x02, J107 Screw_Terminal_01x02, J108 Screw_Terminal_01x02, J109 Screw_Terminal_01x02, J110 282834-4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

Commit message: IDK
Parts:
- moved R116 0.50 mm to (142.0, 19.1)
Routing:
- net +3.3V: track 211.5 -> 260.9 mm
- net DRVOFF: track 283.8 -> 278.0 mm
- net SLEEP_N: track 281.1 -> 275.4 mm
- net Net-(U101-GPIO10/TOUCH10/ADC1_CH9/FSPICS0/FSPIIO4): track 26.7 -> 26.2 mm
